Commit message: Updated boxy urdf and added one without a left arm

File: iai_gazebo_visibility_mover/urdf/boxy_description_transparent_arm.urdf (robot description, URDF)
Before this commit: robot boxy_description, 73 links, 72 joints
Links:
- removed link kinect2_visbility_frame
- link left_arm_1_link: geometry collision mesh filename=package://iai_kuka_lwr4_description/meshes/convex/arm_segme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
- link left_arm_2_link: geometry collision mesh filename=package://iai_kuka_lwr4_description/meshes/convex/arm_segme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
- link left_arm_3_link: geometry collision mesh filename=package://iai_kuka_lwr4_description/meshes/convex/arm_segme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
- link left_arm_4_link: geometry collision mesh filename=package://iai_kuka_lwr4_description/meshes/convex/arm_segme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
- link left_arm_5_link: geometry collision mesh filename=package://iai_kuka_lwr4_description/meshes/convex/arm_segme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
- link left_arm_6_link: geometry collision mesh filename=package://iai_kuka_lwr4_description/meshes/convex/arm_wrist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
- link left_arm_7_link: geometry collision mesh filename=package://iai_kuka_lwr4_description/meshes/convex/arm_flanc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
- link left_arm_cabling_adaptor_link: geometry 
- link left_gripper_base_link: geometry collision mesh filename=package://iai_wsg_50_description/meshes/WSG50_110.stl scale=1 1 1
- link left_gripper_finger_left_link: geometry collision mesh filename=package://iai_wsg_50_description/meshes/WSG-FMF.stl scale=0.001 0.001 0.001
- link left_gripper_finger_right_link: geometry collision mesh filename=package://iai_wsg_50_description/meshes/WSG-FMF.stl scale=0.001 0.001 0.001
- link left_gripper_gripper_left_link: geometry collision mesh filename=package://iai_wsg_50_description/meshes/GUIDE_WSG50_110.stl scale=0.001 0.001 0.001
- link left_gripper_gripper_right_link: geometry collision mesh filename=package://iai_wsg_50_description/meshes/GUIDE_WSG50_110.stl scale=0.001 0.001 0.001
Joints:
- removed joint visibility_joint
